File: Mackie Onyx 1640 USB Option Card/USB_Connector.kicad_sch (KiCad schematic)
At the start: 5 parts, among them J1 USB_B

Commit message: Added a TI-TLV320 ADC Added power for ADC put the filter caps next to pins where they belong Added footprints for ADC and MCU
Parts:
- C1: footprint (none) -> Capacitor_SMD:C_0402_1005Metric
- J2: renamed from J1; footprint (none) -> Connector_USB:USB_B_Lumberg_2411_02_Horizontal
- R1, R2, R3: footprint (none) -> Resistor_SMD:R_0402_1005Metric
Changed lines of the file:
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@@
 			)
 		)
-		(property "Footprint" ""
+		(property "Footprint" "Resistor_SMD:R_0402_1005Metric"
 			(at 115.062 111.76 90)
 			(effects
@@
 		(dnp no)
 		(fields_autoplaced yes)
-		(property "Reference" "J1"
+		(property "Reference" "J2"
 			(at 85.09 97.79 0)
 			(effects
@@
 			)
 		)
-		(property "Footprint" ""
+		(property "Footprint" "Connector_USB:USB_B_Lumberg_2411_02_Horizontal"
 			(at 88.9 111.76 0)
 			(effects
@@
 			(project "Mackie Onyx 1640 USB Option Card"
 				(path "/c9b3cb63-7cfd-4f49-8501-d785ca0cd735/c77f34fa-6c97-4cbe-b773-86889ddd278d"
-					(reference "J1")
+					(reference "J2")
 					(unit 1)
 				)
@@
 			)
 		)
-		(property "Footprint" ""
+		(property "Footprint" "Capacitor_SMD:C_0402_1005Metric"
 			(at 108.9152 115.57 0)
 			(effects
@@
 			)
 		)
-		(property "Footprint" ""
+		(property "Footprint" "Resistor_SMD:R_0402_1005Metric"
 			(at 123.19 107.188 90)
 			(effects
@@
 			)
 		)
-		(property "Footprint" ""
+		(property "Footprint" "Resistor_SMD:R_0402_1005Metric"
 			(at 131.318 111.76 90)
 			(effects
