File: Mackie Onyx 1640 USB Option Card/Connector.kicad_sch (KiCad schematic)
At the start: 1 part, among them J2 Conn_02x17_Odd_Even

Commit message: Added unconnected power pins on connector following firewire-card-schematic
Parts:
- renumbered J2 to J?
Connections:
- net +15V: now also J?.26 (Pin_26)
- net +5V: now also J?.32 (Pin_32), J?.34 (Pin_34)
- net -15V: now also J?.28 (Pin_28)

Commit message: added XMOS XU316-1024-QF60B-C24 MCU (following footprint in pcb) started MCU power and usb phy implementation following datasheet
Parts:
- gave numbers to parts that had none: 1
Changed lines of the file:
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@@
 		(on_board yes)
 		(dnp no)
-		(property "Reference" "J?"
+		(property "Reference" "J2"
 			(at 87.63 24.13 0)
 			(effects
@@
 		(dnp no)
 		(fields_autoplaced yes)
-		(property "Reference" "#PWR03"
+		(property "Reference" "#PWR?"
 			(at 115.57 72.39 0)
 			(effects
@@
 				(path "/a73853a5-305a-4211-9c9e-8d38f21fc90b"
 					(reference "#PWR03")
+					(unit 1)
+				)
+			)
+			(project "Mackie Onyx 1640 USB Option Card"
+				(path "/c9b3cb63-7cfd-4f49-8501-d785ca0cd735/114e7a8f-1ffc-4e4a-996f-c24f2cb4b78c"
+					(reference "#PWR?")
 					(unit 1)
 				)
@@
 		(dnp no)
 		(fields_autoplaced yes)
-		(property "Reference" "#PWR?"
+		(property "Reference" "#PWR09"
 			(at 59.69 72.39 0)
 			(effects
@@
 		(dnp no)
 		(fields_autoplaced yes)
-		(property "Reference" "#PWR?"
+		(property "Reference" "#PWR010"
 			(at 66.04 72.39 0)
 			(effects
@@
 		(dnp no)
 		(fields_autoplaced yes)
-		(property "Reference" "#PWR?"
+		(property "Reference" "#PWR012"
 			(at 78.74 72.39 0)
 			(effects
@@
 		(dnp no)
 		(fields_autoplaced yes)
-		(property "Reference" "#PWR?"
+		(property "Reference" "#PWR08"
 			(at 53.34 82.55 0)
 			(effects
@@
 		(dnp no)
 		(fields_autoplaced yes)
-		(property "Reference" "#PWR01"
+		(property "Reference" "#PWR?"
 			(at 96.52 72.39 0)
 			(effects
@@
 				)
 			)
+			(project "Mackie Onyx 1640 USB Option Card"
+				(path "/c9b3cb63-7cfd-4f49-8501-d785ca0cd735/114e7a8f-1ffc-4e4a-996f-c24f2cb4b78c"
+					(reference "#PWR?")
+					(unit 1)
+				)
+			)
 		)
 	)
@@
 		(dnp no)
 		(fields_autoplaced yes)
-		(property "Reference" "#PWR?"
+		(property "Reference" "#PWR011"
 			(at 72.39 82.55 0)
 			(effects
@@
 		(dnp no)
 		(fields_autoplaced yes)
-		(property "Reference" "#PWR?"
+		(property "Reference" "#PWR014"
 			(at 121.92 82.55 0)
 			(effects
@@
 		(dnp no)
 		(fields_autoplaced yes)
-		(property "Reference" "#PWR?"
+		(property "Reference" "#PWR013"
 			(at 102.87 82.55 0)
 			(effects
@@
 		(dnp no)
 		(fields_autoplaced yes)
-		(property "Reference" "#PWR02"
+		(property "Reference" "#PWR?"
 			(at 109.22 72.39 0)
 			(effects
@@
 					(unit 1)
 				)
+			)
+			(project "Mackie Onyx 1640 USB Option Card"
+				(path "/c9b3cb63-7cfd-4f49-8501-d785ca0cd735/114e7a8f-1ffc-4e4a-996f-c24f2cb4b78c"
+					(reference "#PWR?")
+					(unit 1)
+				)

Commit message: Added a TI-TLV320 ADC Added power for ADC put the filter caps next to pins where they belong Added footprints for ADC and MCU
Parts:
- renumbered J2 to J1
Changed lines of the file:
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@@
 		(on_board yes)
 		(dnp no)
-		(property "Reference" "J2"
+		(property "Reference" "J1"
 			(at 87.63 24.13 0)
 			(effects
@@
 			(project "Mackie Onyx 1640 USB Option Card"
 				(path "/c9b3cb63-7cfd-4f49-8501-d785ca0cd735/114e7a8f-1ffc-4e4a-996f-c24f2cb4b78c"
-					(reference "J2")
+					(reference "J1")
 					(unit 1)
 				)
@@
 		(dnp no)
 		(fields_autoplaced yes)
-		(property "Reference" "#PWR?"
+		(property "Reference" "#PWR0103"
 			(at 115.57 72.39 0)
 			(effects
@@
 			(project "Mackie Onyx 1640 USB Option Card"
 				(path "/c9b3cb63-7cfd-4f49-8501-d785ca0cd735/114e7a8f-1ffc-4e4a-996f-c24f2cb4b78c"
-					(reference "#PWR?")
+					(reference "#PWR0103")
 					(unit 1)
 				)
@@
 		(dnp no)
 		(fields_autoplaced yes)
-		(property "Reference" "#PWR?"
+		(property "Reference" "#PWR0101"
 			(at 96.52 72.39 0)
 			(effects
@@
 			(project "Mackie Onyx 1640 USB Option Card"
 				(path "/c9b3cb63-7cfd-4f49-8501-d785ca0cd735/114e7a8f-1ffc-4e4a-996f-c24f2cb4b78c"
-					(reference "#PWR?")
+					(reference "#PWR0101")
 					(unit 1)
 				)
@@
 		(dnp no)
 		(fields_autoplaced yes)
-		(property "Reference" "#PWR?"
+		(property "Reference" "#PWR0102"
 			(at 109.22 72.39 0)
 			(effects
@@
 			(project "Mackie Onyx 1640 USB Option Card"
 				(path "/c9b3cb63-7cfd-4f49-8501-d785ca0cd735/114e7a8f-1ffc-4e4a-996f-c24f2cb4b78c"
-					(reference "#PWR?")
-					(unit 1)
-				)
+					(reference "#PWR0102")
+					(unit 1)
+				)

Commit message: Added Balancing Circuit ADC input is balanced, card connector isnt schematic following the one from original firewire card since ADC input voltage ratings are very close quad-op-amp-ic is placeholder with standard footprint, a higher quality one may be used on BOM did a bit of more or less rough PCB layouting
Changed lines of the file:
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@@
 	)
 	(hierarchical_label "CH7"
-		(shape input)
+		(shape output)
 		(at 68.58 34.29 180)
 		(effects
@@
 	)
 	(hierarchical_label "CH9"
-		(shape input)
+		(shape output)
 		(at 43.18 36.83 180)
 		(effects
@@
 	)
 	(hierarchical_label "CH1"
-		(shape input)
+		(shape output)
 		(at 43.18 26.67 180)
 		(effects
@@
 	)
 	(hierarchical_label "CH16"
-		(shape input)
+		(shape output)
 		(at 106.68 44.45 0)
 		(effects
@@
 	)
 	(hierarchical_label "CH14"
-		(shape input)
+		(shape output)
 		(at 132.08 41.91 0)
 		(effects
@@
 	)
 	(hierarchical_label "CH2"
-		(shape input)
+		(shape output)
 		(at 132.08 26.67 0)
 		(effects
@@
 	)
 	(hierarchical_label "CH11"
-		(shape input)
+		(shape output)
 		(at 68.58 39.37 180)
 		(effects
@@
 	)
 	(hierarchical_label "CH3"
-		(shape input)
+		(shape output)
 		(at 68.58 29.21 180)
 		(effects
@@
 	)
 	(hierarchical_label "CH4"
-		(shape input)
+		(shape output)
 		(at 106.68 29.21 0)
 		(effects
@@
 	)
 	(hierarchical_label "CH10"
-		(shape input)
+		(shape output)
 		(at 132.08 36.83 0)
 		(effects
@@
 	)
 	(hierarchical_label "CH13"
-		(shape input)
+		(shape output)
 		(at 43.18 41.91 180)
 		(effects
@@
 	)
 	(hierarchical_label "CH12"
-		(shape input)
+		(shape output)
 		(at 106.68 39.37 0)
 		(effects
@@
 	)
 	(hierarchical_label "CH6"
-		(shape input)
+		(shape output)
 		(at 132.08 31.75 0)
 		(effects
@@
 	)
 	(hierarchical_label "CH15"
-		(shape input)
+		(shape output)
 		(at 68.58 44.45 180)
 		(effects
@@
 	)
 	(hierarchical_label "CH5"
-		(shape input)
+		(shape output)
 		(at 43.18 31.75 180)
 		(effects
@@
 	)
 	(hierarchical_label "CH8"
-		(shape input)
+		(shape output)
 		(at 106.68 34.29 0)
 		(effects
