File: Mackie Onyx 1640 USB Option Card/Power_Management.kicad_sch (KiCad schematic)
At the start: 21 parts

Commit message: Added a TI-TLV320 ADC Added power for ADC put the filter caps next to pins where they belong Added footprints for ADC and MCU
Parts:
- added C14, C29: 1uC, Capacitor_SMD:C_0402_1005Metric, symbol Device:C
- added C15, C23, C28, C31: 100nC, Capacitor_SMD:C_0402_1005Metric, symbol Device:C
- added C16, C26, C27, C30: 10uC_Polarized, Capacitor_THT:CP_Radial_D5.0mm_P2.50mm, symbol Device:C_Polarized
- C10, C11, C12, C13, C17, C2, C20, C21, C22, C24, C25, C3, C4, C5, C6, C7, C8, C9: footprint (none) -> Capacitor_SMD:C_0402_1005Metric
- C18, C19: footprint (none) -> Capacitor_THT:CP_Radial_D5.0mm_P2.50mm
- R4: footprint (none) -> Resistor_SMD:R_0402_1005Metric
Connections:
- net +3V3: now also C27.1, C28.2, C30.1, C31.2
- net GND: now also C14.1, C15.1, C16.2, C23.1, C26.2, C27.2, C28.1, C29.1, C30.2, C31.1
- net PLL_AVDD renamed MCU_PLL_AVDD
- new net ADV1_AREG: C15.2, C16.1
- new net ADV1_DREG: C23.2, C26.1
- new net ADV1_MICBIAS: C29.2
- new net ADV1_VREF: C14.2
Other:
- note added: "ADC VDD"
- note added: "trying to follow ADC Datasheet ( https://www.ti.com/lit/ds/symlink/tlv320adc5140.pdf ) Page 108 (Typical Applications)"

Commit message: Added Balancing Circuit ADC input is balanced, card connector isnt schematic following the one from original firewire card since ADC input voltage ratings are very close quad-op-amp-ic is placeholder with standard footprint, a higher quality one may be used on BOM did a bit of more or less rough PCB layouting
Parts:
- removed C16, C26, C27, C30: 10uC_Polarized, Capacitor_THT:CP_Radial_D5.0mm_P2.50mm, symbol Device:C_Polarized
- added C16, C26, C27, C30: 10uC, Capacitor_SMD:C_0805_2012Metric, symbol Device:C
- added C52, C53: 10uC_Polarized, Capacitor_THT:CP_Radial_D4.0mm_P1.50mm, symbol Device:C_Polarized
- C18, C19: footprint Capacitor_THT:CP_Radial_D5.0mm_P2.50mm -> Capacitor_THT:CP_Radial_D4.0mm_P1.50mm
Connections:
- net +3V3: now also C16.2, C27.2
- net ADV1_AREG: now also C30.2
- net ADV1_DREG: now also C26.2
- net GND: now also C16.1, C26.1, C27.1, C30.1, C52.2, C53.1
- new net +15V: C52.1
- new net -15V: C53.2
